File: ICHaus/ICHaus.sch (KiCad schematic (older format))
At the start: 32 parts

Commit message: layout prefinal
Parts:
- added C9: 100n, stmbl:C_0805, symbol stmbl:C
- added D1: LED, LED_SMD:LED_0603_1608Metric, symbol stmbl:LED
- added JP10, JP8, JP9: Jumper_2_Open, Jumper:SolderJumper-2_P1.3mm_Open_RoundedPad1.0x1.5mm, symbol Jumper:Jumper_2_Open
- added JP7: Jumper_2_Bridged, Jumper:SolderJumper-2_P1.3mm_Bridged_RoundedPad1.0x1.5mm, symbol Jumper:Jumper_2_Bridged
- added P1, P2, P3, P4, P5, P6, P7, P8, P9: CONN_01X02, stmbl:RM3.5_1x2, symbol stmbl:CONN_01X02
- added POT1: R_POT, Potentiometer_SMD:Potentiometer_Bourns_3214J_Horizontal, symbol Device:R_POT
- added R8: 220, stmbl:C_0805, symbol stmbl:R
- added RCLK1, ROT1: SolderJumper_3_Open, Jumper:SolderJumper-3_P1.3mm_Bridged12_RoundedPad1.0x1.5mm, symbol Jumper:SolderJumper_3_Bridged12
- added U1, U2, U3, U4: non_plated, stmbl:non_plated_3mm, symbol stmbl:non_plated
- C1, C2, C3, C4, C5, C6, C7, C8: renamed from C?; footprint (none) -> stmbl:C_0805
- J1, J2: renamed from J?; footprint (none) -> Connector_Dsub:DSUB-9_Female_Horizontal_P2.77x2.84mm_EdgePinOffset7.70mm_Housed_MountingHolesOffset9.12mm; symbol Connector:DB9_Female -> Connector:DB9_Female_MountingHoles
- JP1, JP2, JP3: renamed from JP?; footprint (none) -> Jumper:SolderJumper-2_P1.3mm_Open_RoundedPad1.0x1.5mm
- JP4, JP5, JP6: renamed from JP?; footprint (none) -> Jumper:SolderJumper-2_P1.3mm_Bridged_RoundedPad1.0x1.5mm
- PTC1: renamed from PTC?; footprint (none) -> stmbl:C_0805
- R1, R2, R3, R4, R5, R6, R7: renamed from R?; footprint (none) -> stmbl:C_0805
- SF0, SF1, SG0, SG1: renamed from JP?; footprint (none) -> Jumper:SolderJumper-3_P1.3mm_Open_RoundedPad1.0x1.5mm_NumberLabels
- U5: renamed from U?; footprint (none) -> Package_SO:TSSOP-20_4.4x6.5mm_P0.65mm
- U6: renamed from U?; footprint (none) -> Package_SO:SOIC-16_3.9x9.9mm_P1.27mm
- gave numbers to parts that had none: 2
Connections:
- net labels added: A, B, Z
- wire segments 176 -> 227
Other:
- moved on the sheet: C1, C2, C3, C4, C5, C6, C7, C8, JP1, JP2, JP3, JP4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

Commit message: probably final version
Parts:
- added JP11, JP12: SolderJumper_2_Open, Jumper:SolderJumper-2_P1.3mm_Open_RoundedPad1.0x1.5mm, symbol Jumper:SolderJumper_2_Open
- R1: value R -> 120
Connections:
- net +5F: now also JP12.2 (B)
- net GND: now also JP11.2 (B)
- net at C3.1, J1.8, R4.1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: now also P3.1 (P1); no longer P3.2 (P2)
- net at C4.1, J1.7, R6.1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: now also P4.1 (P1), JP12.1 (A); no longer P4.2 (P2)
- net at C4.2, J1.2, JP1.2 (B)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: now also P4.2 (P2), JP11.1 (A); no longer P4.1 (P1)
- net at C2.1, J1.9, R2.1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: now also P2.1 (P1); no longer P2.2 (P2)
- net at C3.2, J1.3, JP2.2 (B)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: now also P3.2 (P2); no longer P3.1 (P1)
- net at C2.2, J1.4, JP3.2 (B)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: now also P2.2 (P2); no longer P2.1 (P1)
Changed lines of the file:
@@
 Connection ~ 3750 3900
 Wire Wire Line
-	3750 4150 4450 4150
+	3750 4150 4100 4150
 Wire Wire Line
 	4450 3750 4450 4150
@@
 P 1700 4450
 F 0 "R1" H 1770 4496 50  0000 L CNN
-F 1 "R" H 1770 4405 50  0000 L CNN
+F 1 "120" H 1770 4405 50  0000 L CNN
 F 2 "stmbl:C_0805" V 1630 4450 50  0001 C CNN
 F 3 "" H 1700 4450 50  0000 C CNN
@@
 F 3 "" H 1200 3350 50  0000 C CNN
 	1    1200 3350
-	-1   0    0    1
+	-1   0    0    -1
 $EndComp
 $Comp
@@
 F 3 "" H 1200 3550 50  0000 C CNN
 	1    1200 3550
-	-1   0    0    1
+	-1   0    0    -1
 $EndComp
 $Comp
@@
 F 3 "" H 1200 3750 50  0000 C CNN
 	1    1200 3750
-	-1   0    0    1
+	-1   0    0    -1
 $EndComp
 $Comp
@@
 	6350 3050 6350 3100
 Connection ~ 6350 3100
+$Comp
+L Jumper:SolderJumper_2_Open JP11
+U 1 1 5EB924C7
+P 2700 4950
+F 0 "JP11" V 2654 5018 50  0000 L CNN
+F 1 "SolderJumper_2_Open" H 2300 4850 50  0000 L CNN
+F 2 "Jumper:SolderJumper-2_P1.3mm_Open_RoundedPad1.0x1.5mm" H 2700 4950 50  0001 C CNN
+F 3 "~" H 2700 4950 50  0001 C CNN
+	1    2700 4950
+	0    1    1    0
+$EndComp
+Wire Wire Line
+	2700 4800 2700 4750
+$Comp
+L power:GND #PWR0111
+U 1 1 5EBA1883
+P 2700 5150
+F 0 "#PWR0111" H 2700 4900 50  0001 C CNN
+F 1 "GND" H 2705 4977 50  0000 C CNN
+F 2 "" H 2700 5150 50  0001 C CNN
+F 3 "" H 2700 5150 50  0001 C CNN
+	1    2700 5150
+	1    0    0    -1
+$EndComp
+Wire Wire Line
+	2700 5100 2700 5150
+$Comp
+L Jumper:SolderJumper_2_Open JP12
+U 1 1 5EBB0393
+P 4100 4350
+F 0 "JP12" V 4054 4418 50  0000 L CNN
+F 1 "SolderJumper_2_Open" H 3700 4250 50  0000 L CNN
+F 2 "Jumper:SolderJumper-2_P1.3mm_Open_RoundedPad1.0x1.5mm" H 4100 4350 50  0001 C CNN
+F 3 "~" H 4100 4350 50  0001 C CNN
+	1    4100 4350
+	0    1    1    0
+$EndComp
+Wire Wire Line
+	4100 4200 4100 4150
+Connection ~ 4100 4150
+Wire Wire Line
+	4100 4150 4450 4150
+$Comp
+L power:+5F #PWR0112
+U 1 1 5EBBF590
+P 4350 4500
+F 0 "#PWR0112" H 4350 4350 50  0001 C CNN
+F 1 "+5F" H 4365 4673 50  0000 C CNN
+F 2 "" H 4350 4500 50  0001 C CNN
+F 3 "" H 4350 4500 50  0001 C CNN
+	1    4350 4500
+	1    0    0    -1
+$EndComp
+Wire Wire Line
+	4100 4500 4100 4550
+Wire Wire Line
+	4100 4550 4350 4550
+Wire Wire Line
+	4350 4550 4350 4500
 $EndSCHEMATC

Commit message: z-detection
added opamp for z impuls detection. (11uass)
Parts:
- removed JP1, JP11: SolderJumper_2_Open, Jumper:SolderJumper-2_P1.3mm_Open_RoundedPad1.0x1.5mm, symbol Jumper:SolderJumper_2_Open
- removed JP6: SolderJumper_2_Bridged, Jumper:SolderJumper-2_P1.3mm_Bridged_RoundedPad1.0x1.5mm, symbol Jumper:SolderJumper_2_Bridged
- added C11: 220p, stmbl:C_0805, symbol stmbl:C
- added JP13, JP14: SolderJumper_2_Open, Jumper:SolderJumper-2_P1.3mm_Open_RoundedPad1.0x1.5mm, symbol Jumper:SolderJumper_2_Open
- added POT2: 50k, Potentiometer_SMD:Potentiometer_Bourns_3214J_Horizontal, symbol Device:R_POT
- added R10: 25k, stmbl:C_0805, symbol stmbl:R
- added R120: 120, stmbl:C_0805, symbol stmbl:R
- added R9: 0, stmbl:C_0805, symbol stmbl:R
- added SG2, SG3: SolderJumper_3_Open, Jumper:SolderJumper-3_P1.3mm_Open_RoundedPad1.0x1.5mm_NumberLabels, symbol Jumper:SolderJumper_3_Open
- added U9: MCP6001U, stmbl:SOIC-8-N, symbol Amplifier_Operational:MCP6002-xSN
- R5: renamed from R1; value 120 -> 220
- R6: renamed from R7; value R -> 100k
- R7: renamed from R6; value R -> 100k
- renumbered C4 to C10, C9 to C8, C8 to C9, R2 to R1, R3 to R2, R4 to R3, R5 to R4
Connections:
- net +5F: now also JP13.2 (B), R10.2, U9.8 (V+); no longer JP12.2 (B)
- net GND: now also POT1.2, JP14.1 (A), R9.1, U9.4 (V-)
- net VREF: now reaches C5.1, JP4.2 (B), JP5.2 (B), U5.5 (VREF)
- net VREF: now also C10.1, R6.2, SG2.3 (B)
- net at R7.2: now also C11.2, SG2.1 (A), U9.2 (-); no longer R6.2
- net at POT1.3, RCLK1.3 (B): no longer POT1.2
- new net: C10.2, R6.1, SG3.1 (A), U9.3 (+)
- new net: C11.1, JP12.2 (B), R7.1, U9.1
- new net: POT2.1, POT2.2, R9.2
- new net VPosIn: JP12.1 (A), JP13.1 (A), SG3.3 (B), U5.17 (P_Zero)
- new net ZNeg: J1.2, P4.2 (P2), R120.2, SG2.2 (C)
- new net ZNegIn: JP14.2 (B), POT2.3, R10.1, U5.18 (N_Zero)
- new net ZPos: J1.7, P4.1 (P1), R120.1, SG3.2 (C)
Other:
- moved on the sheet: C10, C5, R6, R7

Commit message: production files
Parts:
- P1, P2, P3, P4, P5, P6, P7, P8, P9: symbol stmbl:CONN_01X02 -> ICHaus-rescue:CONN_01X02-stmbl
- R5: value 220 -> 120
Changed lines of the file:
@@
 P 1700 4450
 F 0 "R5" H 1770 4496 50  0000 L CNN
-F 1 "220" H 1770 4405 50  0000 L CNN
+F 1 "120" H 1770 4405 50  0000 L CNN
 F 2 "stmbl:C_0805" V 1630 4450 50  0001 C CNN
 F 3 "" H 1700 4450 50  0000 C CNN
@@
 $EndComp
 $Comp
-L stmbl:CONN_01X02 P2
+L ICHaus-rescue:CONN_01X02-stmbl P2
 U 1 1 5ECD6961
 P 1200 3350
@@
 $EndComp
 $Comp
-L stmbl:CONN_01X02 P3
+L ICHaus-rescue:CONN_01X02-stmbl P3
 U 1 1 5ECD807B
 P 1200 3550
@@
 $EndComp
 $Comp
-L stmbl:CONN_01X02 P4
+L ICHaus-rescue:CONN_01X02-stmbl P4
 U 1 1 5ECD84FA
 P 1200 3750
@@
 $EndComp
 $Comp
-L stmbl:CONN_01X02 P1
+L ICHaus-rescue:CONN_01X02-stmbl P1
 U 1 1 5ECD88B1
 P 900 3550
@@
 Connection ~ 2050 3900
 $Comp
-L stmbl:CONN_01X02 P5
+L ICHaus-rescue:CONN_01X02-stmbl P5
 U 1 1 5ED29EC0
 P 1200 4100
@@
 Connection ~ 1500 4050
 $Comp
-L stmbl:CONN_01X02 P6
+L ICHaus-rescue:CONN_01X02-stmbl P6
 U 1 1 5ED6FE16
 P 13050 3650
@@
 $EndComp
 $Comp
-L stmbl:CONN_01X02 P8
+L ICHaus-rescue:CONN_01X02-stmbl P8
 U 1 1 5ED71113
 P 13250 3650
@@
 $EndComp
 $Comp
-L stmbl:CONN_01X02 P9
+L ICHaus-rescue:CONN_01X02-stmbl P9
 U 1 1 5ED71529
 P 13450 3650
@@
 $EndComp
 $Comp
-L stmbl:CONN_01X02 P7
+L ICHaus-rescue:CONN_01X02-stmbl P7
 U 1 1 5ED71881
 P 13250 3400
